File: goya1746.kicad_sch (KiCad schematic)
At the start: 83 parts, among them IC100 TC1044SCPA, IC4 LM2940CT-12_NOPB, J1 GUITAR INPUT, J2 DC INPUT, J3 POWER OUT, J4 GUITAR OUT, U1 OPA2134, U2 TL072, U3 TL072

Commit message: Updated KiCAD v9.0.6. README caps adjustments, updated schematic with buffer and footswich outputs (out of sync with pcb design = not production ready)
Parts:
- added J10: SW4, Connector_Wire:SolderWire-0.5sqmm_1x01_D0.9mm_OD2.1mm, symbol Connector:Conn_01x01_Pin
- added J5: BUFFER, Connector_Wire:SolderWire-0.5sqmm_1x01_D0.9mm_OD2.1mm, symbol Connector:Conn_01x01_Pin
- added J6: SW1, Connector_Wire:SolderWire-0.5sqmm_1x01_D0.9mm_OD2.1mm, symbol Connector:Conn_01x01_Pin
- added J7: SW2, Connector_Wire:SolderWire-0.5sqmm_1x01_D0.9mm_OD2.1mm, symbol Connector:Conn_01x01_Pin
- added J8: GND1, Connector_Wire:SolderWire-0.5sqmm_1x01_D0.9mm_OD2.1mm, symbol Connector:Conn_01x01_Pin
- added J9: SW3, Connector_Wire:SolderWire-0.5sqmm_1x01_D0.9mm_OD2.1mm, symbol Connector:Conn_01x01_Pin
Connections:
- net GND: now also R4.1, J8.1 (Pin_1); no longer D7.2 (Pin_2), R4.2
- net at R17.1, U2.5 (+): now also J7.1 (Pin_1)
- net at C23.1, R36.2, R37.2: now also J9.1 (Pin_1); no longer J4.1 (Pin_1)
- net at C3.2: now also R4.2, J5.1 (Pin_1); no longer R4.1
- new net: J10.1 (Pin_1), J4.1 (Pin_1)
- new net: D7.2 (Pin_2), J6.1 (Pin_1)
Other:
- note added: ""Marshall style" mid-pot tone control. The difference is only with MID pot pins 2 and 3 being connected or not. To switch back to "Fender style" configuration, connect pins 2 and 3 of the MID pot together. P.S: Compare visually with PedalPCB Valhalla Distortion schematic (it's "Fender style" there)"
- note added: "It's a good practice to add 1N5817 Schottky diode between DC Power Jack and DC INPUT pin 1. The striped end (cathode) should face the DC INPUT pin 1."
- note added: "It's either SW1 connected to GND1 when pedal is turned on, or SW2 connected to GND1 when pedal is turned off."
- note added: "POWER OUT is disabled when pedal is turned off. (There won't be any sound) SW4 should be connected to BUFFER when pedal is turned off, or SW3 when pedal is turned on."
- note removed: "1N5817 Schottky diode should be soldered on + wire that leads to DC INPUT (between DC Power Jack and PCB)"
- note removed: "Marshall style mid pot wiring"
- note removed: "TODO: The difference is only with pins 2 and 3 being connected or not. So I would remove this connection for MID & BASS and short it with wires if needed during build process. P.S: Just compare visually with PedalPCB Valhalla Distortion and decide for yourself"
- moved on the sheet: C3, D7, J3, J4, R4
